File: kiCad/RouteEsp32/RouteEsp32.kicad_sch (KiCad schematic)
At the start: 8 parts, among them J1 BAT, J2 ESP32 BAT, J3 GNSS I2C, J4 LCD, U1 MCP23008-xP

Commit message: UT and some schema for PCB
Parts:
- removed J1: BAT, symbol Connector:Conn_01x02_Pin
- removed J2: ESP32 BAT, Connector_JST:JST_PH_B2B-PH-K_1x02_P2.00mm_Vertical, symbol Connector:Conn_01x02_Pin
- removed J3: GNSS I2C, symbol Connector:Conn_01x04_Pin
- removed J4: LCD, symbol Connector:Conn_01x08_Pin
- removed U1: MCP23008-xP, Package_DIP:DIP-18_W7.62mm, symbol Interface_Expansion:MCP23008-xP
- removed uC: Xiao ESP32 S3/C3, Package_DIP:DIP-14_W10.16mm_LongPads, symbol Connector_Generic:Conn_02x07_Counter_Clockwise
- added J1: BAT, Connector_JST:JST_PH_S2B-PH-K_1x02_P2.00mm_Horizontal, symbol Connector_Generic:Conn_01x02
- added J2: ESP32 BAT, Connector_JST:JST_PH_S2B-PH-K_1x02_P2.00mm_Horizontal, symbol Connector_Generic:Conn_01x02
- added J3: GNSS I2C, Connector_JST:JST_PH_S4B-PH-K_1x04_P2.00mm_Horizontal, symbol Connector_Generic:Conn_01x04
- added J4: LCD, Connector_JST:JST_GH_SM08B-GHS-TB_1x08-1MP_P1.25mm_Horizontal, symbol Connector_Generic:Conn_01x08
- added J5: SD Card, Resistor_THT:R_Array_SIP6, symbol Connector_Generic:Conn_01x06
- added J6, J7: BTNS, Connector_PinHeader_2.54mm:PinHeader_1x03_P2.54mm_Horizontal, symbol Connector_Generic:Conn_01x03
- added SW1: prev, Connector_PinHeader_2.54mm:PinHeader_1x02_P2.54mm_Vertical, symbol Switch:SW_MEC_5G
- added SW2: next, Connector_PinHeader_2.54mm:PinHeader_1x02_P2.54mm_Vertical, symbol Switch:SW_MEC_5G
- added U1: XIAO ESP32S3, xiao ESP32C3_PCB:DIP-14_W15.24mm_LongPads, symbol MOUDLE-SEEEDUINO-XIAO-ESP32S3:MOUDLE-SEEEDUINO-XIAO-ESP32S3
- added U3: PCF8574, Package_DIP:DIP-16_W7.62mm, symbol Interface_Expansion:PCF8574
- R1, R2: footprint (none) -> Resistor_THT:R_Axial_DIN0207_L6.3mm_D2.5mm_P2.54mm_Vertical
Connections:
- net GND: now also J3.2 (Pin_2), J4.1 (Pin_1), J6.3 (Pin_3), U1.13 (GND), U3.1 (A0), U3.2 (A1), U3.8 (VSS)
- net BatLvl: now reaches R1.1, R2.1
- net BatLvl: now also U1.1 (PA02_A0_D0)
- net +: now reaches R2.2
- net +: now also J1.1 (Pin_1), J2.1 (Pin_1)
- net -: now reaches R1.2
- net -: now also J1.2 (Pin_2), J2.2 (Pin_2)
- new net: J7.3 (Pin_3), SW1.1 (A), SW1.2 (A), SW2.1 (A), SW2.2 (A)
- new net: J7.1 (Pin_1), SW1.3 (B), SW1.4 (B)
- new net: J7.2 (Pin_2), SW2.3 (B), SW2.4 (B)
- new net +3V3: J3.1 (Pin_1), J4.2 (Pin_2), J5.2 (Pin_2), U1.12 (3V3), U3.16 (VDD), U3.3 (A2)
- new net Btn1: J6.1 (Pin_1), U3.5 (P1)
- new net Btn2: J6.2 (Pin_2), U3.4 (P0)
- new net LCD_BL: J4.8 (Pin_8), U1.4 (PA11_A3_D3)
- new net LCD_CS: J4.5 (Pin_5), U1.8 (PB09_D7_RX)
- new net LCD_DC: J4.6 (Pin_6), U1.2 (PA4_A1_D1)
- new net LCD_RS: J4.7 (Pin_7), U1.3 (PA10_A2_D2)
- new net MISO: J5.3 (Pin_3), U1.10 (PA5_A9_D9_MISO)
- new net MOSI: J4.3 (Pin_3), J5.4 (Pin_4), U1.11 (PA6_A10_D10_MOSI)
- new net SCK: J4.4 (Pin_4), J5.5 (Pin_5), U1.9 (PA7_A8_D8_SCK)
- new net SCL: J3.3 (Pin_3), U1.6 (PA9_A5_D5_SCL), U3.14 (SCL)
- new net SDA: J3.4 (Pin_4), U1.5 (PA8_A4_D4_SDA), U3.15 (SDA)
- new net SD_CS: J5.6 (Pin_6), U1.7 (PB08_A6_TX)
- no-connect marks 3 -> 8
Other:
- title: (none) -> RouteEsp32
- moved on the sheet: R1, R2
